Commit message: 接入激光雷达与 2D SLAM（适配 ROS 2 Jazzy）
==== 一、底层适配 Jazzy（Humble → Jazzy 的差异）====

robot_base_driver：迁移到 hardware_interface 4.48 的新 API。
  - on_init 改用 HardwareComponentInterfaceParams；
  - 不再重写已废弃的 export_state_interfaces()/export_command_interfaces()，
    改由框架按 URDF 自动建接口，驱动用 set_state/get_state/get_command 读写；
  - 句柄在 on_configure（状态）/ on_activate（命令）解析并缓存，控制循环里
    只解引用裸指针，不做 map 查找、不走 wait_until_* 阻塞路径；
  - 位置积分用驱动自有的 hw_positions_，不回读框架的 state 存储
    （后者初值是 NaN，回读会永久污染）。

controllers.yaml：
  - base_frame_id 由 base_link 改为 base_footprint。原先 base_link 同时有
    odom 和 base_footprint 两个父节点，违反 TF「每帧单一父节点」的约束，
    导致树结构非法、base_footprint 整条边被静默丢弃；
  - 移除 Jazzy 已删除的 use_stamped_vel；
  - 新增 position_feedback（Jazzy 新增参数）。

robot_base.launch.py：
  - Jazzy 的 spawner 不再支持 --controller-type/-t，控制器 type 改写入
    参数文件中控制器自己的段；
  - 重映射改走 spawner 的 --controller-ros-args（挂在 controller_manager
    节点上已废弃，运行时会告警）。

view_robot.launch.py：改用专用的 view_robot.rviz
  （robot_base.rviz 已改为建图视图，Fixed Frame 是 map 且无 RobotModel，
   纯可视化时两者都不存在）。

==== 二、激光雷达（YDLIDAR Tmini Pro）====

- 移植 ydlidar_ros2_driver 包，修正上游 launch 里用 LifecycleNode 启动
  普通 Node 的误用，以及会与 URDF 冲突的硬编码静态 TF；
- 新增 udev 规则把雷达绑定为 /dev/ydlidar。CP2102 的序列号是通用值 0001，
  同型号设备全都一样，故用 devpath（USB 物理口编号）区分；
- URDF 新增 laser_frame（挂在 base_link 下），与驱动的 frame_id 参数一致；
- 新增 laser_filters 五级滤波链：
  角度(360°) → 距离截断 → 车体剔除 → 阴影虚点 → 孤立噪点。

==== 三、2D SLAM ====

- slam_toolbox 采用 lifelong（终身建图）模式：会主动淘汰过时节点，
  环境变化时地图持续演化；发布 /map 与 map→odom 的 TF；
- 移植 rf2o_laser_odometry 作激光里程计。robot_base_driver.read() 仍是
  桩实现，轮式里程计不反映真实运动，故 odom 改由雷达提供；
  controllers.yaml 的 enable_odom_tf 相应置 false，避免两个节点
  争抢同一条 odom→base_footprint（会造成 TF 树非法）；
- robot_base.rviz 改为建图视图：Map + /scan_filtered + TF。

==== 实测 ====

雷达 10Hz；滤波后 328 点/帧（滤掉约 7%）；TF 树
map→odom→base_footprint→base_link→laser_frame 完整；
slam_toolbox active；激光里程计漂移与 SLAM 修正量互为逆，
静止时位姿被稳定钉在 map 原点。

注：轮式里程计尚未接真机（read/write 仍是桩实现），
    接好后按 README「接真机后换回轮式里程计」切回。

Co-Authored-By: Claude Code <noreply@anthropic.com>

File: src/robot_base_description/urdf/robot_base.common.xacro (robot description, xacro)
@@ -21,8 +21,12 @@
   <!-- 万向轮（用球体近似） -->
   <xacro:arg name="caster_radius" default="0.02"/>
+  <!-- 激光雷达（YDLIDAR Tmini Pro，用圆柱近似；实际约 70x60mm） -->
+  <xacro:arg name="laser_radius" default="0.035"/>
+  <xacro:arg name="laser_height" default="0.04"/>
   <!-- 质量（kg） -->
   <xacro:arg name="base_mass"   default="8.0"/>
   <xacro:arg name="wheel_mass"  default="0.5"/>
   <xacro:arg name="caster_mass" default="0.1"/>
+  <xacro:arg name="laser_mass"  default="0.15"/>
   <xacro:property name="wheel_radius"     value="$(arg wheel_radius)"/>
   <xacro:property name="wheel_width"      value="$(arg wheel_width)"/>
@@ -32,7 +36,10 @@
   <xacro:property name="base_height"      value="$(arg base_height)"/>
   <xacro:property name="caster_radius"    value="$(arg caster_radius)"/>
+  <xacro:property name="laser_radius"     value="$(arg laser_radius)"/>
+  <xacro:property name="laser_height"     value="$(arg laser_height)"/>
   <xacro:property name="base_mass"        value="$(arg base_mass)"/>
   <xacro:property name="wheel_mass"       value="$(arg wheel_mass)"/>
   <xacro:property name="caster_mass"      value="$(arg caster_mass)"/>
+  <xacro:property name="laser_mass"       value="$(arg laser_mass)"/>
   <!-- ==========================================================================
        惯量宏

File: src/robot_base_description/urdf/robot_base.urdf.xacro (robot description, xacro)
@@ -10,4 +10,5 @@
   <xacro:include filename="$(find robot_base_description)/urdf/robot_base.wheel.xacro"/>
   <xacro:include filename="$(find robot_base_description)/urdf/robot_base.caster.xacro"/>
+  <xacro:include filename="$(find robot_base_description)/urdf/robot_base.lidar.xacro"/>
   <xacro:include filename="$(find robot_base_description)/urdf/robot_base.ros2_control.xacro"/>
   <!-- ==========================================================================
@@ -19,5 +20,6 @@
                ├─ right_wheel_link
                ├─ front_caster_link
-               └─ rear_caster_link
+               ├─ rear_caster_link
+               └─ laser_frame        ← 激光雷达，ydlidar 驱动在此坐标系发 /scan
        ========================================================================== -->
   <link name="base_footprint"/>
@@ -34,4 +36,13 @@
   <xacro:caster prefix="front" reflect="1"  x_offset="${base_length / 2 - caster_radius}"/>
   <xacro:caster prefix="rear"  reflect="-1" x_offset="${base_length / 2 - caster_radius}"/>
+  <!-- 激光雷达。默认认为它坐在底盘顶面正中：
+       底盘顶面在 base_link 的 +base_height/2，雷达光学中心再抬高 半高。
+       ⚠️ 这同样只是占位值，接真机后按实际安装位置改
+          robot_base.lidar.xacro 或被这里的 mount_* 参数覆盖。
+       坐标系名固定为 laser_frame，与 ydlidar 驱动的 frame_id 参数对应。 -->
+  <xacro:lidar prefix="laser"
+               mount_x="0"
+               mount_y="0"
+               mount_z="${base_height / 2 + laser_height / 2}"/>
   <xacro:if value="$(arg use_ros2_control)">
     <xacro:robot_base_ros2_control name="RobotBaseSystem"/>
