Commit message: Add single-lidar navigation, chassis and WeChat bridges

File: src/robot_base_description/urdf/robot_base.ros2_control.xacro (robot description, xacro)
@@ -7,12 +7,26 @@
        ⚠️ 每个关节都必须同时提供 velocity 命令接口和 position+velocity 状态接口，
           否则 RobotBaseSystem::on_init 会直接报错返回。 -->
-  <xacro:macro name="robot_base_ros2_control" params="name">
+  <xacro:macro name="robot_base_ros2_control" params="name use_gazebo:=false">
     <ros2_control name="${name}" type="system">
       <hardware>
-        <!-- 插件名必须与 robot_base_driver.xml 里的 <class name="..."> 完全一致 -->
-        <plugin>robot_base_driver/RobotBaseSystem</plugin>
-        <!-- TODO(hardware): 换成真机的串口设备与波特率 -->
-        <param name="serial_port">/dev/ttyUSB0</param>
-        <param name="baud_rate">115200</param>
+        <xacro:if value="${use_gazebo}">
+          <!-- ================================================================
+               仿真模式：硬件由 Gazebo 提供
+               ================================================================
+               插件类名来自 gz_ros2_control 的 gz_hardware_plugins.xml，
+               它把 Gazebo 里的关节接到 ros2_control 的接口上 ——
+               于是 diff_drive_controller 等控制器**无需任何改动**
+               就能驱动仿真车，这正是 ros2_control 这层抽象的价值。
+               ================================================================ -->
+          <plugin>gz_ros2_control/GazeboSimSystem</plugin>
+        </xacro:if>
+        <xacro:unless value="${use_gazebo}">
+          <!-- 真机模式：走本仓库的串口驱动 -->
+          <!-- 插件名必须与 robot_base_driver.xml 里的 <class name="..."> 完全一致 -->
+          <plugin>robot_base_driver/RobotBaseSystem</plugin>
+          <!-- TODO(hardware): 换成真机的串口设备与波特率 -->
+          <param name="serial_port">/dev/ttyUSB0</param>
+          <param name="baud_rate">115200</param>
+        </xacro:unless>
       </hardware>
       <joint name="left_wheel_joint">

File: src/robot_base_description/urdf/robot_base.urdf.xacro (robot description, xacro)
@@ -1,50 +1,47 @@
 <?xml version="1.0"?>
 <robot name="robot_base" xmlns:xacro="http://www.ros.org/wiki/xacro">
-  <!-- 差速移动机器人底盘 —— 顶层描述文件。
-       common 必须最先 include（它定义后续文件用到的 property 和惯量宏）。 -->
-  <!-- 设为 false 可去掉 <ros2_control> 块：纯可视化时更干净，
-       也便于后续把同一份模型交给 Gazebo（Gazebo 自带硬件接口）。 -->
-  <xacro:arg name="use_ros2_control" default="true"/>
-  <xacro:include filename="$(find robot_base_description)/urdf/robot_base.common.xacro"/>
-  <xacro:include filename="$(find robot_base_description)/urdf/robot_base.base.xacro"/>
-  <xacro:include filename="$(find robot_base_description)/urdf/robot_base.wheel.xacro"/>
-  <xacro:include filename="$(find robot_base_description)/urdf/robot_base.caster.xacro"/>
-  <xacro:include filename="$(find robot_base_description)/urdf/robot_base.lidar.xacro"/>
-  <xacro:include filename="$(find robot_base_description)/urdf/robot_base.ros2_control.xacro"/>
-  <!-- ==========================================================================
-       坐标系约定（REP-103：x 前、y 左、z 上）
-         odom            ← 由 diff_drive_controller 发布
-         └─ base_footprint  地面投影，导航栈常用
-            └─ base_link    底盘几何中心
-               ├─ left_wheel_link
-               ├─ right_wheel_link
-               ├─ front_caster_link
-               ├─ rear_caster_link
-               └─ laser_frame        ← 激光雷达，ydlidar 驱动在此坐标系发 /scan
-       ========================================================================== -->
+  <!-- Preserve the SolidWorks geometry and all four wheel joints. -->
+  <xacro:arg name="use_gazebo" default="false"/>
+  <xacro:include filename="$(find mecanum_car_model)/urdf/mecanum_car_model.urdf"/>
   <link name="base_footprint"/>
   <joint name="base_footprint_joint" type="fixed">
-    <parent link="base_footprint"/>
-    <child link="base_link"/>
-    <!-- 把 base_footprint 放到地面上，即底盘中心抬起 半高+轮半径 -->
-    <origin xyz="0 0 ${base_height / 2 + wheel_radius}" rpy="0 0 0"/>
+    <parent link="base_footprint"/><child link="base_link"/>
+    <origin xyz="0 0 0.069" rpy="0 0 0"/>
   </joint>
-  <xacro:robot_base_base_link/>
-  <!-- reflect=+1 为 +y 侧，即左侧 -->
-  <xacro:wheel prefix="left"  reflect="1"/>
-  <xacro:wheel prefix="right" reflect="-1"/>
-  <xacro:caster prefix="front" reflect="1"  x_offset="${base_length / 2 - caster_radius}"/>
-  <xacro:caster prefix="rear"  reflect="-1" x_offset="${base_length / 2 - caster_radius}"/>
-  <!-- 激光雷达。默认认为它坐在底盘顶面正中：
-       底盘顶面在 base_link 的 +base_height/2，雷达光学中心再抬高 半高。
-       ⚠️ 这同样只是占位值，接真机后按实际安装位置改
-          robot_base.lidar.xacro 或被这里的 mount_* 参数覆盖。
-       坐标系名固定为 laser_frame，与 ydlidar 驱动的 frame_id 参数对应。 -->
-  <xacro:lidar prefix="laser"
-               mount_x="0"
-               mount_y="0"
-               mount_z="${base_height / 2 + laser_height / 2}"/>
-  <xacro:if value="$(arg use_ros2_control)">
-    <xacro:robot_base_ros2_control name="RobotBaseSystem"/>
+  <!-- CAD mesh/wheel maximum XY radius is 0.265 m; allow 35 mm for attachments. -->
+  <link name="navigation_footprint">
+    <visual>
+      <origin xyz="0 0 0" rpy="0 0 0"/>
+      <geometry><cylinder radius="0.30" length="0.01"/></geometry>
+      <material name="navigation_boundary"><color rgba="0.0 0.75 0.85 0.30"/></material>
+    </visual>
+    <!-- Nav2 handles clearance in simulation; an extra Gazebo contact disk would drag on the floor. -->
+    <xacro:unless value="$(arg use_gazebo)">
+      <collision>
+        <origin xyz="0 0 0" rpy="0 0 0"/>
+        <geometry><cylinder radius="0.30" length="0.01"/></geometry>
+      </collision>
+    </xacro:unless>
+  </link>
+  <joint name="navigation_footprint_joint" type="fixed">
+    <parent link="base_footprint"/><child link="navigation_footprint"/>
+    <origin xyz="0 0 0.02" rpy="0 0 0"/>
+  </joint>
+  <!-- CAD front wheels are at -X. Rotate CAD -X onto base_link +X,
+       which is the measured forward direction of laser_frame +Y. -->
+  <link name="base_link"/>
+  <joint name="cad_mount_joint" type="fixed">
+    <parent link="base_link"/><child link="cad_base_link"/>
+    <origin xyz="0 0 0" rpy="0 0 3.141592653589793"/>
+  </joint>
+  <!-- The lidar +Y axis is the confirmed vehicle-forward direction. -->
+  <link name="laser_frame"/>
+  <joint name="laser_joint" type="fixed">
+    <parent link="base_link"/><child link="laser_frame"/>
+    <origin xyz="0.15 0 0.15" rpy="0 0 -1.5707963267948966"/>
+  </joint>
+  <xacro:if value="$(arg use_gazebo)">
+    <xacro:include filename="$(find robot_base_description)/urdf/robot_base.gazebo.xacro"/>
+    <xacro:gazebo_sim/>
   </xacro:if>
 </robot>
