Commit message: 更新麦克纳姆轮小车URDF模型

File: 麦克纳姆轮小车urdf模型文件/mecanum_car_model/urdf/mecanum_car_model.urdf (robot description, URDF)
Before this commit: robot mecanum_car_model, 5 links, 4 joints
Links:
- link Link1: mass 0.056517 -> 0.056517377222027
- link Link3: mass 0.0565173772106941 -> 0.0565173772360903
- link Link4: mass 0.0565173772248273 -> 0.056517377224795
Joints:
- joint wheel_back_left: axis 0 0 1 -> 0 0 0; origin xyz=-0.15175 -0.06721 0.12768 rpy=3.1416 -0.067789 -1.5708 -> xyz=0.16537 -0.1402 0.016148 rpy=-3.1416 0.10332 0
- joint wheel_back_right: axis 0 0 -1 -> 0 0 0; origin xyz=0.12865 -0.06721 0.12768 rpy=3.1416 -0.067789 1.5708 -> xyz=0.16537 0.1402 0.016148 rpy=3.1416 -0.2389 -3.1416
- joint wheel_front_left: axis 0 0 1 -> 0 0 0; origin xyz=-0.13555 0.27094 0.069248 rpy=0 0.54992 -1.5708 -> xyz=-0.17778 -0.124 0.016148 rpy=3.1416 -1.3997 0
- joint wheel_front_right: axis 0 0 -1 -> 0 0 0; origin xyz=0.12865 0.27094 0.069248 rpy=3.1416 0.27443 1.5708 -> xyz=-0.17778 0.1402 0.016148 rpy=3.1416 0.10332 3.1416
