Commit message: 固化实测中生效的配置：footprint 多边形 / 雷达位置 / 代价地图显示
这三处是工作区里一直未提交的改动，本次转向修复的验证就是在它们生效的
状态下跑出来的，所以一并固化，让 main 与"验证通过的那套配置"一致。

1) nav2_params.yaml：两个 costmap 的 robot_radius: 0.30 换成实测的
   整车包络多边形（含四个驱动轮，轮子比车身宽）：
       footprint: "[[-0.2250,-0.1606],[-0.2250,0.1684],[0.2250,0.1684],[0.2250,-0.1606]]"
   长 0.450 m、宽 0.329 m；用 footprint 时不能再写 robot_radius（互斥）。
2) robot_base.urdf.xacro：
   - 雷达移到【前轮轴线】x=0.1716（原 0.15），即左右前轮中心连线上；
     值由 mecanum_car_model.urdf 的前/后轮 x 实测换算得到（x_base = -x_cad - 0.0062），
     并附了推导与交叉校验。
   - cad_mount_joint 的 x=-0.0062 居中平移（让 base_link 落在四轮旋转中心上）及其说明。
3) robot_base.rviz：新增 Global/Local Costmap 显示，并注明为什么 QoS 要用
   Volatile（比 Transient Local 弱，两种发布者都能连上；反过来会完全收不到）。

未改动：功能、参数语义与限幅值都没变，只是把已生效的配置写进版本库。

Co-Authored-By: Claude Code <noreply@anthropic.com>

File: robot_ros2_ws/src/robot_base_description/urdf/robot_base.urdf.xacro (robot description, xacro)
@@ -33,5 +33,14 @@
   <joint name="cad_mount_joint" type="fixed">
     <parent link="base_link"/><child link="cad_base_link"/>
-    <origin xyz="0 0 0" rpy="0 0 3.141592653589793"/>
+    <!-- ⚠️ x=-0.0062 是为了把车体【居中到 base_link 原点】。
+         CAD 导出的模型其几何中心并不在 cad_base_link 原点：实测车身包络中心
+         x=+0.00620、四轮中心 x=+0.00621（两个独立测量互相印证，非网格误差），
+         即旋转中心比原点靠前 6.2mm。base_link 作为运动学中心理应落在旋转中心上，
+         所以这里给一个 -0.0062 的平移把它掰回来。
+         居中后整车包络（base_link 系，含轮子）：
+             x: [-0.2250, +0.2250]   长 0.450 m
+             y: [-0.1606, +0.1684]   宽 0.329 m
+         ⚠️ 本值一旦改动，nav2_params.yaml 里两个 costmap 的 footprint 必须同步重算。 -->
+    <origin xyz="-0.0062 0 0" rpy="0 0 3.141592653589793"/>
   </joint>
   <!-- The lidar +Y axis is the confirmed vehicle-forward direction. -->
@@ -39,5 +48,26 @@
   <joint name="laser_joint" type="fixed">
     <parent link="base_link"/><child link="laser_frame"/>
-    <origin xyz="0.15 0 0.15" rpy="0 0 -1.5707963267948966"/>
+    <!-- ⚠️ 雷达装在【前轮轴线】上，即左前轮与右前轮中心连线的正上方（y=0）。
+         由 CAD 实测（mecanum_car_model.urdf，cad_base_link 系）：
+             前轮 x_cad = -0.17778   （左右两个前轮 x 相同）
+             后轮 x_cad = +0.16537
+         cad_mount_joint 把 CAD 绕 z 转 180° 再平移 -0.0062，故换算到 base_link：
+             x_base = -x_cad - 0.0062
+         前轮：x_base = +0.17778 - 0.0062 = +0.1716   ← 本行取值
+         后轮：x_base = -0.16537 - 0.0062 = -0.1716
+         两轴中点正好落在 0，与"base_link 是四轮旋转中心"的约定自洽，
+         可用来交叉验算（见上方 cad_mount_joint 注释里的 -0.0062）。
+         为什么不放在 0.21：那是贴着车体前缘（包络前沿约 +0.231）装的，
+         雷达本体（半径约 3.5cm）会探出车体约 14mm。移到前轮轴线后雷达
+         完全落在车体内，且与旋转中心的距离更短。
+         ⚠️ 改动本行后需复核两项：
+            1) laser_filters.yaml 的车尾扇区是按【雷达自身】角度定义的，
+               位置变了扇形覆盖的物理区域随之变化；
+            2) 同一文件里 filter2 的 lower_threshold=0.20 是照"雷达扫到
+               自己的安装结构"实测调出来的，挪位置后自回波会变，必要时重测。
+         rpy z=-90°：雷达坐标系相对 base_link 转了 -90°，
+         因此雷达的 +Y 对应 base_link 的 +X。这就是 laser_filters.yaml 里
+         "扫描角 +90° 才是车头方向" 的来源 —— 改动本行前请一并确认那边。 -->
+    <origin xyz="0.1716 0 0.15" rpy="0 0 -1.5707963267948966"/>
   </joint>
   <xacro:if value="$(arg use_gazebo)">
